File: 3dp_esc/3dp_esc/3dp_esc.kicad_pcb (KiCad board)
At the start: 2 copper layers, 32.3 x 29 mm, 16 parts, among them J1 Conn_01x03_Pin, J2 Conn_01x02_Pin, U1 NE555P

Commit message: pinheadersfixed
Parts:
- removed the G*** at (141.1, 131.4)
- J1: footprint Connector_PinHeader_2.00mm:PinHeader_1x03_P2.00mm_Vertical -> Connector_PinHeader_2.54mm:PinHeader_1x03_P2.54mm_Vertical
- J2: footprint Connector_PinHeader_2.00mm:PinHeader_1x02_P2.00mm_Vertical -> Connector_PinHeader_2.54mm:PinHeader_1x02_P2.54mm_Vertical
- moved J1 1.18 mm to (114.3, 119.2)
- moved 1K 0.31 mm to (121.2, 122.5)
Routing:
- net +: track 57.9 -> 50.2 mm
- net -5.6V Bat: track 69.9 -> 72.7 mm
- net Net-(D3-A): track 14.3 -> 15.0 mm
- net signal: track 9.52 -> 10.0 mm

Commit message: i hope its fixed (it isn't)
Parts:
- added 100nF2: C, Capacitor_THT:C_Axial_L3.8mm_D2.6mm_P7.50mm_Horizontal, F.Cu at (11.8, 21.0)
- added 100nf1: C, Capacitor_THT:C_Axial_L3.8mm_D2.6mm_P7.50mm_Horizontal, F.Cu at (11.8, 25.2)
- added 10K1: R_Potentiometer, Potentiometer_THT:Potentiometer_Alps_RK163_Single_Horizontal, F.Cu at (19.1, 4.22)
- added 1K1: R, Resistor_THT:R_Axial_DIN0207_L6.3mm_D2.5mm_P7.62mm_Horizontal, F.Cu at (1.07, 21.0)
- added 220nF1: C, Capacitor_THT:C_Disc_D4.3mm_W1.9mm_P5.00mm, F.Cu at (22.5, 20.7)
- added 68K1: R, Resistor_THT:R_Axial_DIN0207_L6.3mm_D2.5mm_P7.62mm_Horizontal, F.Cu at (1.07, 25.0)
- added D3: LD271, LED_THT:LED_D5.0mm_Clear, F.Cu at (23.4, 26.1)
- J1: footprint Connector_PinHeader_2.54mm:PinHeader_1x03_P2.54mm_Vertical -> Connector_PinHeader_2.00mm:PinHeader_1x03_P2.00mm_Vertical
- J2: footprint Connector_PinHeader_2.54mm:PinHeader_1x02_P2.54mm_Vertical -> Connector_PinHeader_2.00mm:PinHeader_1x02_P2.00mm_Vertical
Connections:
- D2 pad 1: Net-(D2-K) -> jump
- U1 pad 2: Net-(U1-THRES) -> jump
- U1 pad 6: Net-(U1-THRES) -> jump
Routing:
- net Net-(U1-THRES): track 16.1 -> 0.00 mm
- net +: track 50.2 -> 59.5 mm

Commit message: this is good
Parts:
- removed 100nF2, 100nf1: C, Capacitor_THT:C_Axial_L3.8mm_D2.6mm_P7.50mm_Horizontal
- removed 10K: R_Potentiometer, Potentiometer_THT:Potentiometer_Alps_RK163_Single_Horizontal
- removed 1K1, 3K1, 68K1: R, Resistor_THT:R_Axial_DIN0207_L6.3mm_D2.5mm_P7.62mm_Horizontal
- removed 220nF1: C, Capacitor_THT:C_Disc_D4.3mm_W1.9mm_P5.00mm
- removed LED: LD271, LED_THT:LED_D5.0mm_Clear
- added 3K: R, Resistor_THT:R_Axial_DIN0207_L6.3mm_D2.5mm_P7.62mm_Horizontal, F.Cu at (142.7, 118.4)
- moved 10K1 167.5 mm to (136.4, 123.9), turned to 90 degrees
- moved D3 139.7 mm to (136.7, 108.0), turned to 90 degrees
- moved 1uF1 29.1 mm to (153.2, 106.9)
- moved J1 20.3 mm to (134.1, 114.8)
- moved 1K 19.8 mm to (140.6, 118.4)
- moved J2 19.7 mm to (136.2, 111.8)
- moved U1 18.9 mm to (149.4, 108.2)
- moved 100nf 18.5 mm to (141.3, 105.2)
- moved 68K 18.3 mm to (152.9, 119.1)
- moved 100nF 17.5 mm to (156.0, 118.9)
- moved D1 17.0 mm to (159.3, 124.5)
- moved D2 17.0 mm to (159.3, 121.9)
- moved 220nF 16.8 mm to (159.0, 118.8)
- moved G*** 5.29 mm to (145.2, 112.0)
Connections:
- 68K pad 2: Net-(U1-THRES) -> Net-(D2-K)
- D2 pad 1: jump -> Net-(D2-K)
- J2 pad 1: + -> -5.6V Bat
- J2 pad 2: -5.6V Bat -> +
- U1 pad 2: jump -> Net-(D2-K)
- U1 pad 6: jump -> Net-(D2-K)
Routing:
- net Net-(D2-K): track 2.58 -> 29.2 mm
- net -5.6V Bat: track 72.7 -> 47.7 mm
- net +: track 59.5 -> 47.8 mm
- net Net-(D2-A): track 13.5 -> 3.32 mm
- net Net-(D1-K): track 16.8 -> 13.9 mm
- net Net-(10K1-Pad2): track 8.89 -> 5.99 mm
- net signal: track 10.0 -> 9.14 mm
Other:
- board size 32.3 x 29 mm -> 28.7 x 22.8 mm
- board text added: "servo tester"
- board text removed: "3K"
- board text removed: "D1"
